Commit message: Update src

File: src/iai_donbot/iai_donbot_description/robots/iai_donbot.xacro (robot description, xacro)
@@ -1,11 +1,11 @@
 <?xml version="1.0"?>
 <robot xmlns:xacro="http://www.ros.org/wiki/xacro" >
-  <xacro:include filename="$(find iai_donbot)/robots/include/kms_40.urdf.xacro"/>
-  <xacro:include filename="$(find iai_donbot)/robots/include/adapter_fwa050_wsg50.urdf.xacro"/>
-  <xacro:include filename="$(find iai_donbot)/robots/include/adapter_kms40_fwk050.urdf.xacro"/>
-  <xacro:include filename="$(find iai_donbot)/robots/include/fwk_fwa_050.urdf.xacro"/>
-  <xacro:include filename="$(find iai_donbot)/robots/include/ur5.urdf.xacro" />
-  <xacro:include filename="$(find iai_donbot)/robots/iai_donbot_gripper.xacro"/>
-  <xacro:include filename="$(find iai_donbot)/robots/iai_donbot_base.xacro"/>
+  <xacro:include filename="$(find iai_donbot_description)/robots/include/kms_40.urdf.xacro"/>
+  <xacro:include filename="$(find iai_donbot_description)/robots/include/adapter_fwa050_wsg50.urdf.xacro"/>
+  <xacro:include filename="$(find iai_donbot_description)/robots/include/adapter_kms40_fwk050.urdf.xacro"/>
+  <xacro:include filename="$(find iai_donbot_description)/robots/include/fwk_fwa_050.urdf.xacro"/>
+  <xacro:include filename="$(find iai_donbot_description)/robots/include/ur5.urdf.xacro" />
+  <xacro:include filename="$(find iai_donbot_description)/robots/include/iai_donbot_gripper.xacro"/>
+  <xacro:include filename="$(find iai_donbot_description)/robots/include/iai_donbot_base.xacro"/>
   <material name="gray">
     <color rgba="0.56 0.67 0.67 1"/>
@@ -39,5 +39,5 @@
       <visual>
         <geometry>
-          <mesh filename="package://iai_donbot/meshes/iai_table_robot/adapter_plate_iso50_kms40_weiss.stl" scale="0.001 0.001 0.001"/>
+          <mesh filename="package://iai_donbot_description/meshes/iai_table_robot/adapter_plate_iso50_kms40_weiss.stl" scale="0.001 0.001 0.001"/>
         </geometry>
         <material name="gray"/>
@@ -67,5 +67,5 @@
       <visual>
         <geometry>
-          <mesh filename="package://iai_donbot/meshes/iai_refills_camera/refills_camera_holder_and_camera.stl" scale="1 1 1"/>
+          <mesh filename="package://iai_donbot_description/meshes/iai_refills_camera/refills_camera_holder_and_camera.stl" scale="1 1 1"/>
         </geometry>
         <material name="gray"/>
@@ -73,5 +73,5 @@
       <collision>
         <geometry>
-          <mesh filename="package://iai_donbot/meshes/iai_refills_camera/refills_camera_holder_and_camera.stl" scale="1 1 1"/>
+          <mesh filename="package://iai_donbot_description/meshes/iai_refills_camera/refills_camera_holder_and_camera.stl" scale="1 1 1"/>
         </geometry>
         <material name="gray"/>

File: src/iai_donbot/iai_donbot_description/robots/iai_donbot_spawn.xacro (robot description, xacro)
@@ -1,5 +1,5 @@
 <?xml version="1.0"?>
 <robot xmlns:xacro="http://www.ros.org/wiki/xacro" name="iai_donbot">
-  <xacro:include filename="$(find iai_donbot)/robots/iai_donbot.xacro"/>
+  <xacro:include filename="$(find iai_donbot_description)/robots/iai_donbot.xacro"/>
   <xacro:iai_donbot />
   <link name="map">

File: src/iai_donbot/iai_donbot_description/robots/iai_donbot_with_refills_finger_spawn.xacro (robot description, xacro)
@@ -1,5 +1,5 @@
 <?xml version="1.0"?>
 <robot xmlns:xacro="http://www.ros.org/wiki/xacro" name="iai_donbot_with_refills_finger">
-  <xacro:include filename="$(find iai_donbot)/robots/iai_donbot.xacro"/>
+  <xacro:include filename="$(find iai_donbot_description)/robots/iai_donbot.xacro"/>
   <xacro:iai_donbot />
   <joint name="refills_tool_frame_joint" type="fixed">

File: src/iai_donbot/iai_donbot_description/robots/include/adapter_fwa050_wsg50.urdf.xacro (robot description, xacro)
@@ -14,5 +14,5 @@
         <geometry>
           <!-- these meshes were exported in mm, so scale back to m -->
-          <mesh filename="package://iai_donbot/meshes/iai_adapters/adapter_fwa050_wsg50.stl" scale="0.001 0.001 0.001"/>
+          <mesh filename="package://iai_donbot_description/meshes/iai_adapters/adapter_fwa050_wsg50.stl" scale="0.001 0.001 0.001"/>
         </geometry>
         <material name="Grey"/>

File: src/iai_donbot/iai_donbot_description/robots/include/adapter_kms40_fwk050.urdf.xacro (robot description, xacro)
@@ -14,5 +14,5 @@
         <geometry>
           <!-- these meshes were exported in mm, so scale back to m -->
-          <mesh filename="package://iai_donbot/meshes/iai_adapters/adapter_kms40_fwk050.stl" scale="0.001 0.001 0.001"/>
+          <mesh filename="package://iai_donbot_description/meshes/iai_adapters/adapter_kms40_fwk050.stl" scale="0.001 0.001 0.001"/>
         </geometry>
         <material name="Grey"/>

File: src/iai_donbot/iai_donbot_description/robots/include/fwk_fwa_050.urdf.xacro (robot description, xacro)
@@ -14,5 +14,5 @@
         <geometry>
           <!-- these meshes were exported in mm, so scale back to m -->
-          <mesh filename="package://iai_donbot/meshes/iai_adapters/fwk_fwa_050_simple.stl" scale="0.001 0.001 0.001"/>
+          <mesh filename="package://iai_donbot_description/meshes/iai_adapters/fwk_fwa_050_simple.stl" scale="0.001 0.001 0.001"/>
         </geometry>
         <material name="Grey"/>

File: src/iai_donbot/iai_donbot_description/robots/include/iai_donbot_base.xacro (robot description, xacro)
@@ -132,5 +132,5 @@
             <!-- <mesh -->
             <mesh
-            filename="package://iai_donbot/meshes/iai_boxy_base_2/base.stl" />
+            filename="package://iai_donbot_description/meshes/iai_boxy_base_2/base.stl" />
         </geometry>
         <material
@@ -145,5 +145,5 @@
             rpy="0 0 0" />
         <geometry>
-            <mesh filename="package://iai_donbot/meshes/iai_boxy_base_2/base_lowres.stl" />
+            <mesh filename="package://iai_donbot_description/meshes/iai_boxy_base_2/base_lowres.stl" />
         </geometry>
         </collision>

File: src/iai_donbot/iai_donbot_description/robots/include/iai_donbot_gripper.xacro (robot description, xacro)
@@ -17,5 +17,5 @@
             <origin xyz="0.0 0 0" rpy="0 0 0" />
             <geometry>
-                <mesh filename="package://iai_donbot/meshes/iai_wsg_50/WSG50_110.stl" scale="1 1 1"/>
+                <mesh filename="package://iai_donbot_description/meshes/iai_wsg_50/WSG50_110.stl" scale="1 1 1"/>
             </geometry>
             <material name="grey">
@@ -26,5 +26,5 @@
             <origin xyz="0.0 0 0" rpy="0 0 0" />
             <geometry>
-                <mesh filename="package://iai_donbot/meshes/iai_wsg_50/WSG50_110.stl" scale="1 1 1"/>
+                <mesh filename="package://iai_donbot_description/meshes/iai_wsg_50/WSG50_110.stl" scale="1 1 1"/>
             </geometry>
         </collision>
@@ -50,5 +50,5 @@
             <origin xyz="0.0 0 0" rpy="0 0 0" />
             <geometry>
-                <mesh filename="package://iai_donbot/meshes/iai_wsg_50/GUIDE_WSG50_110.stl" scale="0.001 0.001 0.001"/>
+                <mesh filename="package://iai_donbot_description/meshes/iai_wsg_50/GUIDE_WSG50_110.stl" scale="0.001 0.001 0.001"/>
             </geometry>
             <material name="black">
@@ -59,5 +59,5 @@
             <origin xyz="0 0 0" rpy="0 0 0" />
             <geometry>
-                <mesh filename="package://iai_donbot/meshes/iai_wsg_50/GUIDE_WSG50_110.stl" scale="0.001 0.001 0.001"/>
+                <mesh filename="package://iai_donbot_description/meshes/iai_wsg_50/GUIDE_WSG50_110.stl" scale="0.001 0.001 0.001"/>
             </geometry>
         </collision>
@@ -82,5 +82,5 @@
             <origin xyz="0.0 0 0" rpy="0 0 0" />
             <geometry>
-                <mesh filename="package://iai_donbot/meshes/iai_wsg_50/WSG-FMF.stl" scale="0.001 0.001 0.001"/>
+                <mesh filename="package://iai_donbot_description/meshes/iai_wsg_50/WSG-FMF.stl" scale="0.001 0.001 0.001"/>
             </geometry>
             <material name="black">
@@ -91,5 +91,5 @@
             <origin xyz="0 0 0" rpy="0 0 0" />
             <geometry>
-                <mesh filename="package://iai_donbot/meshes/iai_wsg_50/WSG-FMF.stl" scale="0.001 0.001 0.001"/>
+                <mesh filename="package://iai_donbot_description/meshes/iai_wsg_50/WSG-FMF.stl" scale="0.001 0.001 0.001"/>
             </geometry>
         </collision>
@@ -116,5 +116,5 @@
             <origin xyz="0.0 0 0" rpy="0 0 0" />
             <geometry>
-                <mesh filename="package://iai_donbot/meshes/iai_wsg_50/GUIDE_WSG50_110.stl" scale="0.001 0.001 0.001"/>
+                <mesh filename="package://iai_donbot_description/meshes/iai_wsg_50/GUIDE_WSG50_110.stl" scale="0.001 0.001 0.001"/>
             <!--box size="0.0175 0.03 0.024"/-->
             </geometry>
@@ -127,5 +127,5 @@
             <geometry>
             <!--box size="0.0175 0.03 0.024"/-->
-                <mesh filename="package://iai_donbot/meshes/iai_wsg_50/GUIDE_WSG50_110.stl" scale="0.001 0.001 0.001"/>
+                <mesh filename="package://iai_donbot_description/meshes/iai_wsg_50/GUIDE_WSG50_110.stl" scale="0.001 0.001 0.001"/>
             </geometry>
         </collision>
@@ -148,5 +148,5 @@
             <origin xyz="0.0 0 0" rpy="0 0 0" />
             <geometry>
-                <mesh filename="package://iai_donbot/meshes/iai_wsg_50/WSG-FMF.stl" scale="0.001 0.001 0.001"/>
+                <mesh filename="package://iai_donbot_description/meshes/iai_wsg_50/WSG-FMF.stl" scale="0.001 0.001 0.001"/>
             </geometry>
             <material name="black">
@@ -157,5 +157,5 @@
             <origin xyz="0 0 0" rpy="0 0 0" />
             <geometry>
-                <mesh filename="package://iai_donbot/meshes/iai_wsg_50/WSG-FMF.stl" scale="0.001 0.001 0.001"/>
+                <mesh filename="package://iai_donbot_description/meshes/iai_wsg_50/WSG-FMF.stl" scale="0.001 0.001 0.001"/>
             </geometry>
         </collision>

File: src/iai_donbot/iai_donbot_description/robots/include/kms_40.urdf.xacro (robot description, xacro)
@@ -14,5 +14,5 @@
         <origin rpy="0 0 0" xyz="0 0 0"/>
         <geometry>
-          <mesh filename="package://iai_donbot/meshes/iai_kms_40/adapter_plate_iso50_kms40_weiss.stl" scale="0.001 0.001 0.001"/>
+          <mesh filename="package://iai_donbot_description/meshes/iai_kms_40/adapter_plate_iso50_kms40_weiss.stl" scale="0.001 0.001 0.001"/>
         </geometry>
         <material name="Grey"/>
@@ -39,5 +39,5 @@
         <origin rpy="0 0 0" xyz="0 0 0"/>
         <geometry>
-          <mesh filename="package://iai_donbot/meshes/iai_kms_40/kms40_simple.stl" scale="0.001 0.001 0.001"/>
+          <mesh filename="package://iai_donbot_description/meshes/iai_kms_40/kms40_simple.stl" scale="0.001 0.001 0.001"/>
         </geometry>
         <material name="Grey"/>

File: src/iai_donbot/iai_donbot_description/robots/include/ur5.urdf.xacro (robot description, xacro)
@@ -73,13 +73,13 @@
       <visual>
         <geometry>
-          <mesh filename="package://iai_donbot/meshes/ur5/visual/base.dae" />
-        </geometry>
-        <material name="LightGrey">
-          <color rgba="0.7 0.7 0.7 1.0"/>
-        </material>
-      </visual>
-      <collision>
-        <geometry>
-          <mesh filename="package://iai_donbot/meshes/ur5/collision/base.stl" />
+          <mesh filename="package://iai_donbot_description/meshes/ur5/visual/base.dae" />
+        </geometry>
+        <material name="LightGrey">
+          <color rgba="0.7 0.7 0.7 1.0"/>
+        </material>
+      </visual>
+      <collision>
+        <geometry>
+          <mesh filename="package://iai_donbot_description/meshes/ur5/collision/base.stl" />
         </geometry>
       </collision>
@@ -104,13 +104,13 @@
       <visual>
         <geometry>
-          <mesh filename="package://iai_donbot/meshes/ur5/visual/shoulder.dae" />
-        </geometry>
-        <material name="LightGrey">
-          <color rgba="0.7 0.7 0.7 1.0"/>
-        </material>
-      </visual>
-      <collision>
-        <geometry>
-          <mesh filename="package://iai_donbot/meshes/ur5/collision/shoulder.stl" />
+          <mesh filename="package://iai_donbot_description/meshes/ur5/visual/shoulder.dae" />
+        </geometry>
+        <material name="LightGrey">
+          <color rgba="0.7 0.7 0.7 1.0"/>
+        </material>
+      </visual>
+      <collision>
+        <geometry>
+          <mesh filename="package://iai_donbot_description/meshes/ur5/collision/shoulder.stl" />
         </geometry>
       </collision>
@@ -135,13 +135,13 @@
       <visual>
         <geometry>
-          <mesh filename="package://iai_donbot/meshes/ur5/visual/upperarm.dae" />
-        </geometry>
-        <material name="LightGrey">
-          <color rgba="0.7 0.7 0.7 1.0"/>
-        </material>
-      </visual>
-      <collision>
-        <geometry>
-          <mesh filename="package://iai_donbot/meshes/ur5/collision/upperarm.stl" />
+          <mesh filename="package://iai_donbot_description/meshes/ur5/visual/upperarm.dae" />
+        </geometry>
+        <material name="LightGrey">
+          <color rgba="0.7 0.7 0.7 1.0"/>
+        </material>
+      </visual>
+      <collision>
+        <geometry>
+          <mesh filename="package://iai_donbot_description/meshes/ur5/collision/upperarm.stl" />
         </geometry>
       </collision>
@@ -166,13 +166,13 @@
       <visual>
         <geometry>
-          <mesh filename="package://iai_donbot/meshes/ur5/visual/forearm.dae" />
-        </geometry>
-        <material name="LightGrey">
-          <color rgba="0.7 0.7 0.7 1.0"/>
-        </material>
-      </visual>
-      <collision>
-        <geometry>
-          <mesh filename="package://iai_donbot/meshes/ur5/collision/forearm.stl" />
+          <mesh filename="package://iai_donbot_description/meshes/ur5/visual/forearm.dae" />
+        </geometry>
+        <material name="LightGrey">
+          <color rgba="0.7 0.7 0.7 1.0"/>
+        </material>
+      </visual>
+      <collision>
+        <geometry>
+          <mesh filename="package://iai_donbot_description/meshes/ur5/collision/forearm.stl" />
         </geometry>
       </collision>
@@ -197,13 +197,13 @@
       <visual>
         <geometry>
-          <mesh filename="package://iai_donbot/meshes/ur5/visual/wrist1.dae" />
-        </geometry>
-        <material name="LightGrey">
-          <color rgba="0.7 0.7 0.7 1.0"/>
-        </material>
-      </visual>
-      <collision>
-        <geometry>
-          <mesh filename="package://iai_donbot/meshes/ur5/collision/wrist1.stl" />
+          <mesh filename="package://iai_donbot_description/meshes/ur5/visual/wrist1.dae" />
+        </geometry>
+        <material name="LightGrey">
+          <color rgba="0.7 0.7 0.7 1.0"/>
+        </material>
+      </visual>
+      <collision>
+        <geometry>
+          <mesh filename="package://iai_donbot_description/meshes/ur5/collision/wrist1.stl" />
         </geometry>
       </collision>
@@ -228,13 +228,13 @@
       <visual>
         <geometry>
-          <mesh filename="package://iai_donbot/meshes/ur5/visual/wrist2.dae" />
-        </geometry>
-        <material name="LightGrey">
-          <color rgba="0.7 0.7 0.7 1.0"/>
-        </material>
-      </visual>
-      <collision>
-        <geometry>
-          <mesh filename="package://iai_donbot/meshes/ur5/collision/wrist2.stl" />
+          <mesh filename="package://iai_donbot_description/meshes/ur5/visual/wrist2.dae" />
+        </geometry>
+        <material name="LightGrey">
+          <color rgba="0.7 0.7 0.7 1.0"/>
+        </material>
+      </visual>
+      <collision>
+        <geometry>
+          <mesh filename="package://iai_donbot_description/meshes/ur5/collision/wrist2.stl" />
         </geometry>
       </collision>
@@ -259,13 +259,13 @@
       <visual>
         <geometry>
-          <mesh filename="package://iai_donbot/meshes/ur5/visual/wrist3.dae" />
-        </geometry>
-        <material name="LightGrey">
-          <color rgba="0.7 0.7 0.7 1.0"/>
-        </material>
-      </visual>
-      <collision>
-        <geometry>
-          <mesh filename="package://iai_donbot/meshes/ur5/collision/wrist3.stl" />
+          <mesh filename="package://iai_donbot_description/meshes/ur5/visual/wrist3.dae" />
+        </geometry>
+        <material name="LightGrey">
+          <color rgba="0.7 0.7 0.7 1.0"/>
+        </material>
+      </visual>
+      <collision>
+        <geometry>
+          <mesh filename="package://iai_donbot_description/meshes/ur5/collision/wrist3.stl" />
         </geometry>
       </collision>

File: src/iai_donbot/iai_donbot_gazebo/robots/iai_donbot_gazebo.xacro (robot description, xacro)
@@ -1,10 +1,10 @@
 <?xml version="1.0"?>
 <robot xmlns:xacro="http://wiki.ros.org/xacro" name="iai_donbot">
-    <xacro:include filename="$(find iai_donbot)/robots/iai_donbot.xacro"/>
+    <xacro:include filename="$(find iai_donbot_description)/robots/iai_donbot.xacro"/>
     <xacro:iai_donbot />
-    <xacro:include filename="$(find iai_donbot)/robots/iai_donbot.transmission.xacro"/>
+    <xacro:include filename="$(find iai_donbot_gazebo)/robots/iai_donbot.transmission.xacro"/>
     <xacro:ur_arm_transmission prefix="ur5_"/>
     <!-- Load joint controller configurations from YAML file to parameter server -->
-    <rosparam file="$(find iai_donbot)/config/iai_donbot_control.yaml" command="load"/>
+    <rosparam file="$(find iai_donbot_gazebo)/config/iai_donbot_control.yaml" command="load"/>
     <gazebo reference="">
         <plugin name="gazebo_ros_control" filename="libgazebo_ros_control.so">
