Commit message: Update iai_donbot_unreal

File: src/iai_donbot/iai_donbot_description/urdf/iai_donbot_spawn.xacro (robot description, xacro)
@@ -1,6 +1,6 @@
 <?xml version="1.0"?>
 <robot xmlns:xacro="http://www.ros.org/wiki/xacro" name="iai_donbot">
-  <xacro:include filename="$(find iai_donbot_description)/robots/iai_donbot.xacro"/>
-  <xacro:iai_donbot />
+  <xacro:include filename="$(find iai_donbot_description)/urdf/iai_donbot.xacro"/>
+  <xacro:include filename="$(find iai_donbot_description)/urdf/include/iai_donbot_odom.xacro"/>
   <link name="map">
     </link>

File: src/iai_donbot/iai_donbot_description/urdf/iai_donbot_with_refills_finger_spawn.xacro (robot description, xacro)
@@ -1,6 +1,5 @@
 <?xml version="1.0"?>
-<robot xmlns:xacro="http://www.ros.org/wiki/xacro" name="iai_donbot_with_refills_finger">
-  <xacro:include filename="$(find iai_donbot_description)/robots/iai_donbot.xacro"/>
-  <xacro:iai_donbot />
+<robot xmlns:xacro="http://www.ros.org/wiki/xacro" name="iai_donbot">
+  <xacro:include filename="$(find iai_donbot_description)/urdf/iai_donbot_spawn.xacro"/>
   <joint name="refills_tool_frame_joint" type="fixed">
     <parent link="gripper_tool_frame"/>

File: src/iai_donbot/iai_donbot_description/urdf/include/iai_donbot_base.xacro (robot description, xacro)
@@ -1,74 +1,3 @@
 <robot name="base">
-    <link name="odom">
-        <inertial>
-            <origin xyz="0.0 0.0 0.0" rpy="0.0 0.0 0.0"/>
-            <mass value="1E-4"/>
-            <inertia ixx="1E-4" ixy="0.0" ixz="0.0" iyy="1E-4" iyz="0.0" izz="1E-4"/>
-        </inertial>
-        <visual>
-            <origin rpy="0 0 0" xyz="0 0 0"/>
-            <geometry>
-            <box size="0.01 0.01 0.01"/>
-            </geometry>
-            <material name="White"/>
-        </visual>
-    </link>
-    <joint name="odom_x_joint" type="prismatic">
-        <parent link="odom"/>
-        <child link="odom_x_frame"/>
-        <axis xyz="1 0 0"/>
-        <!-- limits chosen heuristically
-            lower/upper: +-1km to create a quasi limitless prismatic joint
-            velocity: slow walking speed is 3-4km/hour ~= 1m/s
-            effort: reach max speed within 1s, Boxy has a mass of 200kg, so Fmax=200kg*1m/s2 -->
-        <limit lower="-1000" upper="1000" velocity="1" effort="20000"/>
-    </joint>
-    <link name="odom_x_frame">
-        <inertial>
-            <origin xyz="0.0 0.0 0.0" rpy="0.0 0.0 0.0"/>
-            <mass value="1E-4"/>
-            <inertia ixx="1E-4" ixy="0.0" ixz="0.0" iyy="1E-4" iyz="0.0" izz="1E-4"/>
-        </inertial>
-        <visual>
-            <origin rpy="0 0 0" xyz="0 0 0"/>
-            <geometry>
-            <box size="0.01 0.01 0.01"/>
-            </geometry>
-            <material name="White"/>
-        </visual>
-    </link>
-    <joint name="odom_y_joint" type="prismatic">
-        <parent link="odom_x_frame"/>
-        <child link="odom_y_frame"/>
-        <axis xyz="0 1 0"/>
-        <!-- limits chosen heuristically
-            lower/upper: +-1km to create a quasi limitless prismatic joint
-            velocity: slow walking speed is 3-4km/hour ~= 1m/s
-            effort: reach max speed within 1s, Boxy has a mass of 200kg, so Fmax=200kg*1m/s2 -->
-        <limit lower="-1000" upper="1000" velocity="1" effort="20000"/>
-    </joint>
-    <link name="odom_y_frame">
-        <inertial>
-            <origin xyz="0.0 0.0 0.0" rpy="0.0 0.0 0.0"/>
-            <mass value="1E-4"/>
-            <inertia ixx="1E-4" ixy="0.0" ixz="0.0" iyy="1E-4" iyz="0.0" izz="1E-4"/>
-        </inertial>
-        <visual>
-            <origin rpy="0 0 0" xyz="0 0 0"/>
-            <geometry>
-            <box size="0.01 0.01 0.01"/>
-            </geometry>
-            <material name="White"/>
-        </visual>
-    </link>
-    <joint name="odom_z_joint" type="continuous">
-        <parent link="odom_y_frame"/>
-        <child link="base_footprint"/>
-        <axis xyz="0 0 1"/>
-        <!-- limits chosen heuristically
-            velocity: one slow complete turn around in 5-6s, so 6.2rad/6s ~= 1rad/s
-            effort: reach max speed within 1s, Boxy has a mass of 200kg and a diagonale of 1m, so Fmax=200kg*1m*1m/s2 -->
-        <limit velocity="1" effort="20000"/>
-    </joint>
     <!-- Definition of base_footprint -> base_link -->
     <link name="base_footprint">

File: src/iai_donbot/iai_donbot_gazebo/urdf/iai_donbot_gazebo.xacro (robot description, xacro)
@@ -1,7 +1,7 @@
 <?xml version="1.0"?>
 <robot xmlns:xacro="http://wiki.ros.org/xacro" name="iai_donbot">
-    <xacro:include filename="$(find iai_donbot_description)/robots/iai_donbot.xacro"/>
-    <xacro:iai_donbot />
-    <xacro:include filename="$(find iai_donbot_gazebo)/robots/iai_donbot.transmission.xacro"/>
+    <xacro:include filename="$(find iai_donbot_description)/urdf/iai_donbot.xacro"/>
+    <xacro:include filename="$(find iai_donbot_description)/urdf/include/iai_donbot_odom.xacro"/>
+    <xacro:include filename="$(find iai_donbot_gazebo)/urdf/iai_donbot.transmission.xacro"/>
     <xacro:ur_arm_transmission prefix="ur5_"/>
     <!-- Load joint controller configurations from YAML file to parameter server -->
