Commit message: Update donbot

File: src/iai_donbot/iai_donbot_description/urdf/iai_donbot.xacro (robot description, xacro)
@@ -82,5 +82,11 @@
     <origin xyz="0 0 0" rpy="0 0 ${pi}" />
   </joint>
-  <link name="camera_link"/>
+  <link name="camera_link">
+    <visual>
+      <geometry>
+        <cylinder radius="0.001" length="0.005"/>
+      </geometry>
+    </visual>
+  </link>
   <joint name="gripper_to_camera_joint" type="fixed">
     <parent link="gripper_base_link" />

File: src/iai_donbot/iai_donbot_unreal/iai_donbot_unreal/urdf/iai_donbot_unreal.urdf (robot description, URDF)
Before this commit: robot iai_donbot, 41 links, 40 joints
Links:
- link camera_link: geometry visual cylinder length=0.005 radius=0.001

File: src/iai_donbot/iai_donbot_unreal/iai_donbot_unreal/urdf/iai_donbot_unreal.xacro (robot description, xacro)
@@ -4,3 +4,8 @@
   <!--Add odom-->
   <xacro:include filename="$(find iai_donbot_description)/urdf/include/iai_donbot_odom.xacro"/>
+  <link name="map"/>
+  <joint name="map_link" type="fixed">
+    <parent link="map"/>
+    <child link="odom"/>
+  </joint>
 </robot>
