Commit message: Update iai_donbot

File: src/iai_donbot/iai_donbot_description/urdf/include/iai_donbot_base.xacro (robot description, xacro)
@@ -10,8 +10,14 @@
             <origin rpy="0 0 0" xyz="0 0 0"/>
             <geometry>
-            <box size="0.01 0.01 0.01"/>
+                <box size="0.01 0.01 0.01"/>
             </geometry>
             <material name="White"/>
         </visual>
+        <collision>
+            <origin rpy="0 0 0" xyz="0 0 0"/>
+            <geometry>
+                <box size="0.01 0.01 0.01"/>
+            </geometry>
+        </collision>
     </link>
     <!-- JOINT to define base_footprint -->
@@ -121,5 +127,4 @@
         </collision>
     </link>
-    <!-- JOINT to define base_footprint -->
     <joint name="plate_joint" type="fixed">
         <origin xyz="-0.300 -0.230 0.460" rpy="0 0 0" />

File: src/iai_donbot/iai_donbot_unreal/iai_donbot_unreal/urdf/iai_donbot_unreal.urdf (robot description, URDF)
Before this commit: robot iai_donbot, 41 links, 40 joints
Links:
- link base_footprint: geometry collision box size=0.01 0.01 0.01; visual box size=0.01 0.01 0.01

File: src/iai_donbot/iai_donbot_unreal/iai_donbot_unreal/urdf/iai_donbot_unreal.xacro (robot description, xacro)
@@ -5,5 +5,5 @@
   <xacro:include filename="$(find iai_donbot_description)/urdf/include/iai_donbot_odom.xacro"/>
   <link name="map"/>
-  <joint name="map_link" type="fixed">
+  <joint name="map_joint" type="fixed">
     <parent link="map"/>
     <child link="odom"/>
