Commit message: Change gripper joint orientation

File: src/iai_donbot/iai_donbot_description/urdf/include/iai_donbot_gripper.xacro (robot description, xacro)
@@ -32,10 +32,10 @@
     <!-- GRIPPER LEFT -->
     <joint name="${name}_base_gripper_left_joint" type="prismatic">
-        <limit lower="-0.051" upper="0" effort="10.0" velocity="0.42"/>
+        <limit lower="0" upper="0.051" effort="10.0" velocity="0.42"/>
         <origin xyz="-0.0040 0 0" rpy="0 0 0" />
         <parent link="${name}_base_link"/>
         <child link="${name}_gripper_left_link" />
         <dynamics friction="1" damping="1" />
-        <axis xyz="1 0 0"/>
+        <axis xyz="-1 0 0"/>
     </joint>
     <link name="${name}_gripper_left_link">

File: src/iai_donbot/iai_donbot_unreal/iai_donbot_unreal/urdf/iai_donbot_unreal.urdf (robot description, URDF)
Before this commit: robot iai_donbot, 41 links, 40 joints
Joints:
- joint gripper_base_gripper_left_joint: axis 1 0 0 -> -1 0 0; limit lower=-0.051 upper=0 effort=10.0 velocity=0.42 -> lower=0 upper=0.051 effort=10.0 velocity=0.42
