Commit message: Add navigation

File: src/iai_donbot/iai_donbot_gazebo/urdf/iai_donbot_gazebo.xacro (robot description, xacro)
@@ -53,4 +53,13 @@
         </sensor>
     </gazebo>
+    <joint name="hokuyo_joint" type="fixed">
+        <axis xyz="0 1 0" />
+        <origin xyz="0 0 0" rpy="0 0 0"/>
+        <parent link="laser_reference_front"/>
+        <child link="hokuyo_link"/>
+    </joint>
+    <!-- Hokuyo Laser -->
+    <link name="hokuyo_link">
+    </link>
     <link name="world">
     </link>
@@ -60,3 +69,39 @@
         <child link="odom"/>
     </joint>
+    <!-- hokuyo -->
+    <gazebo reference="hokuyo_link">
+        <sensor type="gpu_ray" name="head_hokuyo_sensor">
+        <pose>0 0 0 0 0 0</pose>
+        <visualize>false</visualize>
+        <update_rate>40</update_rate>
+        <ray>
+            <scan>
+            <horizontal>
+                <samples>720</samples>
+                <resolution>1</resolution>
+                <min_angle>-1.570796</min_angle>
+                <max_angle>1.570796</max_angle>
+            </horizontal>
+            </scan>
+            <range>
+            <min>0.10</min>
+            <max>30.0</max>
+            <resolution>0.01</resolution>
+            </range>
+            <noise>
+            <type>gaussian</type>
+            <!-- Noise parameters based on published spec for Hokuyo laser
+                achieving "+-30mm" accuracy at range < 10m.  A mean of 0.0m and
+                stddev of 0.01m will put 99.7% of samples within 0.03m of the true
+                reading. -->
+            <mean>0.0</mean>
+            <stddev>0.01</stddev>
+            </noise>
+        </ray>
+        <plugin name="gazebo_ros_head_hokuyo_controller" filename="libgazebo_ros_gpu_laser.so">
+            <topicName>/iai_donbot/laser/scan</topicName>
+            <frameName>hokuyo_link</frameName>
+        </plugin>
+        </sensor>
+    </gazebo>
 </robot>

File: src/iai_donbot/iai_donbot_unreal/iai_donbot_unreal/urdf/iai_donbot_unreal.xacro (robot description, xacro)
@@ -4,8 +4,3 @@
   <!--Add odom-->
   <xacro:include filename="$(find iai_donbot_description)/urdf/include/iai_donbot_odom.xacro"/>
-  <link name="map"/>
-  <joint name="map_joint" type="fixed">
-    <parent link="map"/>
-    <child link="odom"/>
-  </joint>
 </robot>
