Commit message: Add amcl, navigation

File: src/iai_donbot/iai_donbot_unreal/iai_donbot_unreal/urdf/iai_donbot_unreal.xacro (robot description, xacro)
@@ -4,3 +4,10 @@
   <!--Add odom-->
   <xacro:include filename="$(find iai_donbot_description)/urdf/include/iai_donbot_odom.xacro"/>
+  <!--link name="map">
+  </link>
+  <joint name="map_joint" type="fixed">
+    <origin xyz="0.0 0.0 0.0" rpy="0.0 0.0 0.0"/>
+    <parent link="map"/>
+    <child link="odom"/>
+  </joint-->
 </robot>
